File: TM4C129 Breakout_Hardware/TM4C129-Breakout_Hardware.kicad_pcb (KiCad board)
At the start: 2 copper layers, 63.5 x 47 mm, 50 parts, among them J1 RJ45, J2 Conn_02x08, J3 Conn_02x08, J4 Conn_02x08, J5 Conn_02x02, J6 Conn_02x02, SW1 SW_Push, U1 HX1198FNL, U2 TM4C129ENCPDT, Y1 NX3225GA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

Commit message: fixed headers to go down
Parts:
- J2, J3, J4, J5, J6: moved to B.Cu
- moved J5 2.54 mm to (132.1, 30.5), turned to 180 degrees
- moved J6 2.54 mm to (149.9, 30.5), turned to 180 degrees
- moved J2 2.54 mm to (109.2, 30.5), turned to 180 degrees
- moved J3 2.54 mm to (109.2, 53.3), turned to 180 degrees
- moved J4 2.54 mm to (165.1, 30.5), turned to 180 degrees
Connections:
- J2 pad 1: A0 -> A8
- J2 pad 10: A12 -> A4
- J2 pad 11: A5 -> A13
- J2 pad 12: A13 -> A5
- J2 pad 13: A6 -> A14
- J2 pad 14: A14 -> A6
- J2 pad 15: A7 -> A15
- J2 pad 16: A15 -> A7
- J2 pad 2: A8 -> A0
- J2 pad 3: A1 -> A9
- J2 pad 4: A9 -> A1
- J2 pad 5: A2 -> A10
- J2 pad 6: A10 -> A2
- J2 pad 7: A3 -> A11
- J2 pad 8: A11 -> A3
- J2 pad 9: A4 -> A12
- J3 pad 1: RX0 -> TX0
- J3 pad 10: TX4 -> RX4
- J3 pad 11: RX5 -> TX5
- J3 pad 12: TX5 -> RX5
- J3 pad 13: RX6 -> TX6
- J3 pad 14: TX6 -> RX6
- J3 pad 15: RX7 -> TX7
- J3 pad 16: TX7 -> RX7
- J3 pad 2: TX0 -> RX0
- J3 pad 3: RX1 -> TX1
- J3 pad 4: TX1 -> RX1
- J3 pad 5: RX2 -> TX2
- J3 pad 6: TX2 -> RX2
- J3 pad 7: RX3 -> TX3
- J3 pad 8: TX3 -> RX3
- J3 pad 9: RX4 -> TX4
- J4 pad 1: Net-(J4-Pad1) -> T2_A
- J4 pad 10: T4_A -> PWM4
- J4 pad 11: PWM5 -> T4_B
- J4 pad 12: T4_B -> PWM5
- J4 pad 13: PWM6 -> T5_A
- J4 pad 14: T5_A -> PWM6
- J4 pad 15: PWM7 -> T5_B
- J4 pad 16: T5_B -> PWM7
- J4 pad 2: T2_A -> Net-(J4-Pad2)
- J4 pad 3: PWM1 -> T2_B
- J4 pad 4: T2_B -> PWM1
- J4 pad 5: PWM2 -> T3_A
- J4 pad 6: T3_A -> PWM2
- J4 pad 7: PWM3 -> T3_B
- J4 pad 8: T3_B -> PWM3
- J4 pad 9: PWM4 -> T4_A
- J5 pad 1: +3V3 -> GND
- J5 pad 2: GND -> +3V3
- J5 pad 3: SDA0 -> SCL0
- J5 pad 4: SCL0 -> SDA0
- J6 pad 1: +3V3 -> GND
- J6 pad 2: GND -> +3V3
- J6 pad 3: +3V3 -> GND
- J6 pad 4: GND -> +3V3
Routing:
- net A9: track 30.6 -> 31.2 mm
- net A10: track 39.1 -> 39.6 mm
Other:
- board text added: "TM4C129 Breakout, Rev 1 Mars Rover Design Team Missouri S&T, 2020 Andrew Van Horn"
- board text removed: "TM4C129 Breakout Mars Rover Design Team Missouri S&T, 2020 Andrew Van Horn"

Commit message: fixed changes before PRR
Parts:
- added C19: 12p, Capacitor_SMD:C_0603_1608Metric_Pad1.05x0.95mm_HandSolder, F.Cu at (135.6, 38.0)
- moved R16 10.9 mm to (149.5, 62.0)
- moved R17 9.40 mm to (149.5, 51.8)
- moved R10 2.79 mm to (149.5, 57.9)
- moved R9 1.27 mm to (149.5, 55.9)
- moved R7 0.76 mm to (149.5, 53.8)
- moved R8 0.76 mm to (149.5, 59.9)
Connections:
- Conn1 pad 10: RST -> ~RST
- J1 pad 10: Ethernet_Link -> Ethernet_Activity
- J1 pad 12: Ethernet_Activity -> Ethernet_Link
- J1 pad 2: Net-(J1-Pad1) -> Net-(J1-Pad2)
- J1 pad 8: Net-(J1-Pad8) -> Net-(J1-Pad7)
- R10 pad 2: Net-(J1-Pad1) -> Net-(J1-Pad7)
- R16 pad 1: Net-(J1-Pad9) -> Net-(J1-Pad11)
- R17 pad 1: Net-(J1-Pad11) -> Net-(J1-Pad9)
- U1 pad 11: Net-(J1-Pad6) -> Net-(J1-Pad3)
- U1 pad 14: Net-(J1-Pad7) -> Net-(J1-Pad2)
- U1 pad 16: Net-(J1-Pad8) -> Net-(J1-Pad1)
- U1 pad 9: Net-(J1-Pad3) -> Net-(J1-Pad6)
Routing:
- net ~RST: track 10.3 -> 104.5 mm, vias 0 -> 2
- net Net-(J1-Pad8): track 28.2 -> 0.00 mm, vias 1 -> 0
- net Net-(J1-Pad2): track 0.00 -> 22.7 mm, vias 0 -> 1
- net Net-(J1-Pad7): track 33.1 -> 13.1 mm
- net Net-(J1-Pad1): track 10.2 -> 23.0 mm, vias 0 -> 1
- net Net-(J1-Pad3): track 35.1 -> 29.2 mm
- net Ethernet_Link: track 32.4 -> 27.2 mm
- net Net-(R8-Pad2): track 17.4 -> 14.8 mm
- net Ethernet_Activity: track 27.2 -> 29.5 mm
- net Net-(J1-Pad6): track 25.2 -> 22.9 mm, vias 2 -> 0
- net Net-(C19-Pad2): track 2.12 -> 3.82 mm
- net GND: track 30.4 -> 31.7 mm, vias 10 -> 48
- net Net-(R7-Pad2): track 15.2 -> 14.0 mm
- net Net-(J1-Pad4): track 10.2 -> 10.8 mm, vias 0 -> 1

Commit message: Minor Aesthetic changes
Parts:
- renumbered SW1 to Reset
Routing:
- net +3V3: track 135.3 -> 129.9 mm
Changed lines of the file:
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@@
     (thickness 1.6)
     (drawings 20)
-    (tracks 1129)
+    (tracks 1124)
     (zones 0)
     (modules 51)
@@
   (module MRDT_Devices:HX1198FNL (layer F.Cu)
     (at 144.272 74.549 90)
-    (fp_text reference U1 (at 10.668 1.4224 90) (layer F.SilkS)
+    (fp_text reference U1 (at 0.635 1.016 180) (layer F.SilkS)
       (effects (font (size 1 1) (thickness 0.15)))
     )
@@
     (tags "TL3305 Series Tact Switch")
     (attr smd)
-    (fp_text reference SW1 (at -0.972 3.024 180) (layer F.SilkS)
+    (fp_text reference Reset (at 0.044 3.024 180) (layer F.SilkS)
       (effects (font (size 1 1) (thickness 0.15)))
     )
@@
   (segment (start 134.119879 65.031879) (end 134.119879 70.858121) (width 0.762) (layer B.Cu) (net 2))
   (via (at 122.174 71.12) (size 0.8) (drill 0.4) (layers F.Cu B.Cu) (net 2))
-  (segment (start 122.174 70.104) (end 122.174 71.12) (width 0.2286) (layer F.Cu) (net 2))
   (segment (start 122.174 70.104) (end 121.158 70.104) (width 0.2286) (layer F.Cu) (net 2))
   (segment (start 123.218 70.104) (end 122.174 70.104) (width 0.2286) (layer F.Cu) (net 2))
@@
   (segment (start 129.794 72.136) (end 130.838 72.136) (width 0.2286) (layer F.Cu) (net 2))
   (segment (start 128.778 72.136) (end 129.794 72.136) (width 0.2286) (layer F.Cu) (net 2))
-  (segment (start 122.174 72.136) (end 122.174 71.12) (width 0.2286) (layer F.Cu) (net 2))
   (segment (start 122.174 72.136) (end 121.158 72.136) (width 0.2286) (layer F.Cu) (net 2))
   (segment (start 123.218 72.136) (end 122.174 72.136) (width 0.2286) (layer F.Cu) (net 2))
-  (segment (start 123.218 71.12) (end 121.158 71.12) (width 0.2286) (layer F.Cu) (net 2))
   (segment (start 121.158 71.12) (end 121.158 72.136) (width 0.2286) (layer F.Cu) (net 2))
   (segment (start 121.158 70.104) (end 121.158 71.12) (width 0.2286) (layer F.Cu) (net 2))
@@
   (segment (start 123.218 70.104) (end 123.218 71.12) (width 0.2286) (layer F.Cu) (net 2))
   (segment (start 122.174 71.12) (end 133.858 71.12) (width 0.762) (layer B.Cu) (net 2))
-  (via (at 143.002 48.006) (size 0.8) (drill 0.4) (layers F.Cu B.Cu) (net 2))
+  (via (at 143.002 48.768) (size 0.8) (drill 0.4) (layers F.Cu B.Cu) (net 2))
   (segment (start 119.634 46.764843) (end 119.634 46.736) (width 0.2286) (layer F.Cu) (net 2))
   (segment (start 120.143856 47.274699) (end 119.634 46.764843) (width 0.2286) (layer F.Cu) (net 2))
@@
   (segment (start 141.224 47.978) (end 141.196 48.006) (width 0.381) (layer F.Cu) (net 2))
   (segment (start 141.196 48.006) (end 143.002 48.006) (width 0.381) (layer F.Cu) (net 2))
-  (segment (start 143.51 48.006) (end 143.002 48.006) (width 0.381) (layer B.Cu) (net 2))
-  (segment (start 143.764 48.26) (end 143.51 48.006) (width 0.381) (layer B.Cu) (net 2))
-  (segment (start 143.764 52.832) (end 143.764 48.26) (width 0.381) (layer B.Cu) (net 2))
   (segment (start 141.6685 54.8005) (end 140.97 54.102) (width 0.762) (layer F.Cu) (net 2))
   (segment (start 141.6685 55.372) (end 141.6685 54.8005) (width 0.762) (layer F.Cu) (net 2))
@@
   (segment (start 138.684 54.102) (end 136.906 52.324) (width 0.762) (layer F.Cu) (net 2))
   (segment (start 140.97 54.102) (end 138.684 54.102) (width 0.762) (layer F.Cu) (net 2))
-  (segment (start 140.97 54.102) (end 143.256 54.102) (width 0.381) (layer B.Cu) (net 2))
-  (segment (start 143.764 53.594) (end 143.764 52.832) (width 0.381) (layer B.Cu) (net 2))
-  (segment (start 143.256 54.102) (end 143.764 53.594) (width 0.381) (layer B.Cu) (net 2))
   (segment (start 143.002 48.006) (end 144.752 48.006) (width 0.381) (layer F.Cu) (net 2))
   (segment (start 144.752 48.006) (end 144.78 47.978) (width 0.381) (layer F.Cu) (net 2))
+  (segment (start 143.002 53.594) (end 142.494 54.102) (width 0.381) (layer B.Cu) (net 2))
+  (segment (start 143.002 48.768) (end 143.002 53.594) (width 0.381) (layer B.Cu) (net 2))
+  (segment (start 140.97 54.102) (end 142.494 54.102) (width 0.381) (layer B.Cu) (net 2))
+  (segment (start 143.002 48.768) (end 143.002 48.006) (width 0.381) (layer F.Cu) (net 2))
   (segment (start 142.494 73.152) (end 143.002 73.66) (width 0.381) (layer F.Cu) (net 3))
   (segment (start 143.002 73.66) (end 149.606 73.66) (width 0.381) (layer F.Cu) (net 3))
@@
       )
     )
+  )
+  (zone (net 2) (net_name +3V3) (layer F.Cu) (hatch edge 0.508)
+    (priority 1)
+    (connect_pads yes (clearance 0.1524))
+    (min_thickness 0.254)
+    (fill yes (arc_segments 16) (thermal_gap 0.508) (thermal_bridge_width 0.508))
+    (polygon
+      (pts
+        (xy 121.158 70.104) (xy 123.19 70.104) (xy 123.19 72.136) (xy 121.158 72.136)
+      )
+    )
+  )
+  (zone (net 2) (net_name +3V3) (layer F.Cu) (hatch edge 0.508)
+    (priority 1)
+    (connect_pads yes (clearance 0.1524))
+    (min_thickness 0.254)
+    (fill yes (arc_segments 16) (thermal_gap 0.508) (thermal_bridge_width 0.508))
+    (polygon
+      (pts
+        (xy 128.806 70.104) (xy 130.838 70.104) (xy 130.838 72.136) (xy 128.806 72.136)
+      )
+    )

Commit message: Final changes before PRR
Routing:
- net +3V3: track 129.9 -> 109.4 mm, vias 11 -> 15

Commit message: Revert "Revert "Merge branch 'master' of https://github.com/MissouriMRDT/TM4C129-Breakout_Hardware""
This reverts commit 4686fe645caf3e9fbf8c00f0c0ea95986b0ea6b8.
Parts:
- C14: value .1uF -> 1uF
- SW1: renamed from Reset; value SW_Push -> Reset
Connections:
- R1 pad 2: EN0RXI_N -> EN0TXO_P
- R2 pad 2: EN0RXI_P -> EN0TXO_N
- R3 pad 2: EN0TXO_N -> EN0RXI_P
- R4 pad 2: EN0TXO_P -> EN0RXI_N
- U1 pad 1: EN0RXI_N -> EN0TXO_P
- U1 pad 3: EN0RXI_P -> EN0TXO_N
- U1 pad 6: EN0TXO_N -> EN0RXI_P
- U1 pad 8: EN0TXO_P -> EN0RXI_N
Routing:
- net +3V3: track 109.4 -> 121.3 mm, vias 15 -> 14
- net EN0TXO_N: track 22.9 -> 31.9 mm, vias 0 -> 2
- net EN0RXI_P: track 29.0 -> 23.1 mm, vias 0 -> 2
- net Ethernet_Link: track 27.2 -> 31.2 mm
- net EN0TXO_P: track 26.6 -> 29.8 mm, vias 0 -> 2
- net Ethernet_Activity: track 29.5 -> 27.7 mm
- net EN0RXI_N: track 25.0 -> 26.0 mm, vias 0 -> 2
- net GND: vias 48 -> 49
- added copper zone on B.Cu, net (none)
- added copper zone on F.Cu, net (none)
Other:
- board text added: "Reset"

Commit message: Revert "Merge branch 'master' of https://github.com/MissouriMRDT/TM4C129-Breakout_Hardware"
This reverts commit e6cd920ed13198a4f7d11fd6171e0ba52050bff9, reversing
changes made to e15dd7d36717f2d892901729c8f3941fb424f385.
Parts:
- C14: value 1uF -> .1uF
- Reset: renamed from SW1; value Reset -> SW_Push
Connections:
- R1 pad 2: EN0TXO_P -> EN0RXI_N
- R2 pad 2: EN0TXO_N -> EN0RXI_P
- R3 pad 2: EN0RXI_P -> EN0TXO_N
- R4 pad 2: EN0RXI_N -> EN0TXO_P
- U1 pad 1: EN0TXO_P -> EN0RXI_N
- U1 pad 3: EN0TXO_N -> EN0RXI_P
- U1 pad 6: EN0RXI_P -> EN0TXO_N
- U1 pad 8: EN0RXI_N -> EN0TXO_P
Routing:
- net +3V3: track 121.3 -> 109.4 mm, vias 14 -> 15
- net EN0TXO_N: track 31.9 -> 22.9 mm, vias 2 -> 0
- net EN0RXI_P: track 23.1 -> 29.0 mm, vias 2 -> 0
- net Ethernet_Link: track 31.2 -> 27.2 mm
- net EN0TXO_P: track 29.8 -> 26.6 mm, vias 2 -> 0
- net Ethernet_Activity: track 27.7 -> 29.5 mm
- net EN0RXI_N: track 26.0 -> 25.0 mm, vias 2 -> 0
- net GND: vias 49 -> 48
- removed copper zone on B.Cu, net (none)
- removed copper zone on F.Cu, net (none)
Other:
- board text removed: "Reset"
