File: TM4C129 Breakout_Hardware/TM4C129-Breakout_Hardware.kicad_pcb (KiCad board)
At the start: 2 copper layers, 63.5 x 47 mm, 54 parts, among them J1 RJ45, J2 Conn_02x08, J3 Conn_02x08, J4 Conn_02x08, J5 Conn_02x02, J6 Conn_02x02, SW1 Reset, U1 HX1198FNL, U2 TM4C129ENCPDT, Y1 NX3225GA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

Commit message: Created Rev3 Gerbs
Parts:
- removed the G*** at (45.7, 16.5)
- moved G*** 153.9 mm to (147.8, 105.2)
Other:
- board text removed: "TM4C129 Breakout, Rev 2 Mars Rover Design Team Missouri S&T, 2020 Andrew Van Horn"
